File: hardware/Croí - Kicad/Croí.kicad_sch (KiCad schematic)
At the start: 38 parts, among them J1 JTAG-10 PIN, J2 2060-1452/998-404, J3 ESQ-110-14-G-D, Q1 IPP060N06N, U1 W25Q128JVS, U2 ADXL375BCCZ, U3 STM32F072C8Tx, U4 BME680, U5 BMP390, U7 TLV70433DBVT, U8 TJA1051T-3, U9 LSM6DSO32TR

Commit message: crazy work
Parts:
- removed J2: 2060-1452/998-404, footprints:WAG, symbol wago:2060-1452_998-404
Other:
- moved on the sheet: Q1
Changed lines of the file:
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@@
 	)
 	(junction
-		(at 157.48 123.19)
-		(diameter 0)
-		(color 0 0 0 0)
-	)
-	(junction
 		(at 205.74 45.72)
 		(diameter 0)
@@
 	)
 	(junction
-		(at 154.94 130.81)
-		(diameter 0)
-		(color 0 0 0 0)
-	)
-	(junction
 		(at 280.67 38.1)
 		(diameter 0)
@@
 	(wire
 		(pts
-			(xy 154.94 130.81) (xy 157.48 130.81)
-		)
-		(stroke
-			(width 0)
-			(type default)
-		)
-	)
-	(wire
-		(pts
 			(xy 280.67 24.13) (xy 280.67 29.21)
 		)
@@
 	(wire
 		(pts
-			(xy 154.94 128.27) (xy 154.94 130.81)
-		)
-		(stroke
-			(width 0)
-			(type default)
-		)
-	)
-	(wire
-		(pts
 			(xy 97.79 53.34) (xy 97.79 50.8)
 		)
@@
 	(wire
 		(pts
-			(xy 157.48 128.27) (xy 154.94 128.27)
-		)
-		(stroke
-			(width 0)
-			(type default)
-		)
-	)
-	(wire
-		(pts
 			(xy 161.29 205.74) (xy 158.75 205.74)
 		)
@@
 	(wire
 		(pts
-			(xy 157.48 123.19) (xy 157.48 125.73)
-		)
-		(stroke
-			(width 0)
-			(type default)
-		)
-	)
-	(wire
-		(pts
 			(xy 205.74 45.72) (xy 213.36 45.72)
 		)
@@
 	(global_label "VBAT"
 		(shape input)
-		(at 147.32 123.19 270)
+		(at 154.94 127 270)
 		(fields_autoplaced yes)
 		(effects
@@
 		)
 		(property "Intersheetrefs" "${INTERSHEET_REFS}"
-			(at 147.32 130.59 90)
+			(at 154.94 134.4 90)
 			(effects
 				(font
@@
 	(symbol
 		(lib_id "power:GND")
-		(at 154.94 130.81 0)
+		(at 205.74 127 90)
 		(unit 1)
 		(exclude_from_sim no)
@@
 		(fields_autoplaced yes)
 		(property "Reference" "#PWR012"
-			(at 154.94 137.16 0)
+			(at 212.09 127 0)
 			(effects
 				(font
@@
 		)
 		(property "Value" "GND"
-			(at 154.94 135.89 0)
+			(at 209.55 126.9999 90)
 			(effects
 				(font
 					(size 1.27 1.27)
 				)
+				(justify right)
 			)
 		)
 		(property "Footprint" ""
-			(at 154.94 130.81 0)
+			(at 205.74 127 0)
 			(effects
 				(font
@@
 		)
 		(property "Datasheet" ""
-			(at 154.94 130.81 0)
+			(at 205.74 127 0)
 			(effects
 				(font
@@
 		)
 		(property "Description" "Power symbol creates a global label with name \"GND\" , ground"
-			(at 154.94 130.81 0)
+			(at 205.74 127 0)
 			(effects
 				(font
@@
 	(symbol
 		(lib_id "Transistor_FET:IPP060N06N")
-		(at 152.4 120.65 270)
+		(at 160.02 124.46 270)
 		(unit 1)
 		(exclude_from_sim no)
@@
 		(fields_autoplaced yes)
 		(property "Reference" "Q1"
-			(at 152.4 127 90)
+			(at 160.02 130.81 90)
 			(effects
 				(font
@@
 		)
 		(property "Value" "IPP060N06N"
-			(at 152.4 129.54 90)
+			(at 160.02 133.35 90)
 			(effects
 				(font
@@
 		)
 		(property "Footprint" "Package_TO_SOT_THT:TO-220-3_Vertical"
-			(at 150.495 125.73 0)
+			(at 158.115 129.54 0)
 			(effects
 				(font
@@
 		)
 		(property "Datasheet" "https://www.infineon.com/dgdl/Infineon-IPP060N06N-DS-v02_02-en.pdf?fileId=db3a30433727a44301372c06d9d7498a"
-			(at 148.59 125.73 0)
+			(at 156.21 129.54 0)
 			(effects
 				(font
@@
 		)
 		(property "Description" "45A Id, 60V Vds, Single N-Channel Power MOSFET, 6mOhm Ron, TO-220"
-			(at 152.4 120.65 0)
+			(at 160.02 124.46 0)
 			(effects
 				(font
@@
 	(symbol
 		(lib_id "power:GND")
-		(at 152.4 115.57 180)
+		(at 160.02 119.38 180)
 		(unit 1)
 		(exclude_from_sim no)
@@
 		(fields_autoplaced yes)
 		(property "Reference" "#PWR08"
-			(at 152.4 109.22 0)
+			(at 160.02 113.03 0)
 			(effects
 				(font
@@
 		)
 		(property "Value" "GND"
-			(at 152.4 110.49 0)
+			(at 160.02 114.3 0)
 			(effects
 				(font
@@
 		)
 		(property "Footprint" ""
-			(at 152.4 115.57 0)
+			(at 160.02 119.38 0)
 			(effects
 				(font
@@
 		)
 		(property "Datasheet" ""
-			(at 152.4 115.57 0)
+			(at 160.02 119.38 0)
 			(effects
 				(font
@@
 		)
 		(property "Description" "Power symbol creates a global label with name \"GND\" , ground"
-			(at 152.4 115.57 0)
+			(at 160.02 119.38 0)
 			(effects
 				(font
@@
 					(unit 1)
 				)
-			)
-		)
-	)
-	(symbol
-		(lib_id "wago:2060-1452_998-404")
-		(at 157.48 123.19 0)
-		(unit 1)
-		(exclude_from_sim no)
-		(in_bom yes)
-		(on_board yes)
-		(dnp no)
-		(fields_autoplaced yes)
-		(property "Reference" "J2"
-			(at 171.45 125.7299 0)
-			(effects
-				(font
-					(size 1.524 1.524)
-				)
-				(justify left)
-			)
-		)
-		(property "Value" "2060-1452/998-404"
-			(at 171.45 128.2699 0)
-			(effects
-				(font
-					(size 1.524 1.524)
-				)
-				(justify left)
-			)
-		)
-		(property "Footprint" "footprints:WAG"
-			(at 157.48 123.19 0)
-			(effects
-				(font
-					(size 1.27 1.27)
-					(italic yes)
-				)
-				(hide yes)
-			)
-		)
-		(property "Datasheet" "2060-1452/998-404"
-			(at 157.48 123.19 0)
-			(effects
-				(font
-					(size 1.27 1.27)
-					(italic yes)
-				)
-				(hide yes)
-			)
-		)
-		(property "Description" ""
-			(at 157.48 123.19 0)
-			(effects
-				(font
-					(size 1.27 1.27)
-				)
-				(hide yes)
-			)
-		)
-		(pin "4"
-		)
-		(pin "2"
-		)
-		(pin "1"
-		)
-		(pin "3"
-		)
-		(instances
-			(project "Croí"
-				(path "/c72f7211-c022-4e45-b2e6-f28a82a66d95"
-					(reference "J2")
-					(unit 1)
-				)

Commit message: Board Routing completed: Ready for Review
Parts:
- added J2: XT30PW-M, footprints:AMASS_XT30PW-M, symbol XT30PW-M:XT30PW-M
Connections:
- net GND: now also J2.N
- net at Q1.2 (D): now also J2.P
Other:
- moved on the sheet: Q1
