File: hardware/Croí - Kicad/Croí.kicad_sch (KiCad schematic)
At the start: 46 parts, among them J1 5023860570, J2 39-29-1048, J3 ESQ-110-14-G-D, Q1 IPD90P04P4L04ATMA1, U1 W25Q128JVS, U2 ADXL375BCCZ, U3 STM32F072C8Tx, U4 BME680, U5 BMP390, U8 TJA1051T-3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

Commit message: clean asf
Parts:
- U9: footprint footprints:LGA-14L_2P5X3X0P83_STM -> LGA-14L_2P5X3X0P83_STM
Connections:
- net 5V_LOGIC is gone; now on net 5VLOGIC: D1.2
- net SWCLK2 is gone; now on net SWCLK: U3.37 (PA14)
- net VBAT_Local is gone; now on net VBAT: D1.1
Changed lines of the file:
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@@
 		)
 	)
-	(global_label "SWCLK2"
+	(global_label "SWCLK"
 		(shape input)
 		(at 116.84 96.52 0)
@@
 		)
 		(property "Intersheetrefs" "${INTERSHEET_REFS}"
-			(at 127.2637 96.52 0)
+			(at 126.0542 96.52 0)
 			(effects
 				(font
@@
 		)
 	)
-	(global_label "5V_LOGIC"
+	(global_label "5VLOGIC"
 		(shape input)
 		(at 250.825 24.13 0)
@@
 		)
 		(property "Intersheetrefs" "${INTERSHEET_REFS}"
-			(at 262.5793 24.13 0)
+			(at 261.6117 24.13 0)
 			(effects
 				(font
@@
 		)
 	)
-	(global_label "VBAT_Local"
+	(global_label "VBAT"
 		(shape input)
 		(at 233.045 24.13 0)
@@
 		)
 		(property "Intersheetrefs" "${INTERSHEET_REFS}"
-			(at 246.4925 24.13 0)
+			(at 240.445 24.13 0)
 			(effects
 				(font
@@
 			)
 		)
-		(property "Footprint" "footprints:LGA-14L_2P5X3X0P83_STM"
+		(property "Footprint" "LGA-14L_2P5X3X0P83_STM"
 			(at 156.21 172.72 0)
 			(effects

Commit message: good to go
Parts:
- removed C18, C20: 100nF, Capacitor_SMD:C_0402_1005Metric, symbol Device:C
- removed U5: BMP390, footprints:10LGA_2X2X0p75_BOS, symbol BMP390:BMP390
- added C48: 100nF, Resistor_SMD:R_0402_1005Metric, symbol Device:C
- added U12: MS560702BA03-50, SON125P300X500X100-8N, symbol MS560702BA03-50:MS560702BA03-50
Connections:
- net 3.3V: now also C48.2, U12.1 (VDD)
- net GND: now also C48.1, U12.2 (PS), U12.3 (GND)
- net SPICLK: now also U12.8 (SCLK)
- net SPI_MISO: now also U12.6 (SDO)
- net SPI_MOSI: now also U12.7 (SDI/SDA)
- net BMP390_CS renamed SPI_CS_MS5
- net SPI_CS_MS5: now also U12.4 (~{CSB}), U12.5 (~{CSB})
- no-connect marks 32 -> 31
Other:
- moved on the sheet: 3V3, C19, D1, GND1, U4

Commit message: progress, not flashing yet
Parts:
- added D3: 1N4148W, Diode_SMD:D_SOD-123, symbol Diode:1N4148W
- added LS1: AT-1224-TWT-12V-2-R, XDCR_AT-1224-TWT-12V-2-R, symbol AT-1224-TWT-12V-2-R:AT-1224-TWT-12V-2-R
- added Q5: AO3400A, Package_TO_SOT_SMD:SOT-23, symbol Transistor_FET:AO3400A
- added R5: 10KΩ, Resistor_SMD:R_0402_1005Metric, symbol Device:R
- added R8: 1KΩ, Resistor_SMD:R_0402_1005Metric, symbol Device:R
- C12, C24, C26: footprint Capacitor_SMD:C_0402_1005Metric -> Capacitor_SMD:C_0603_1608Metric
Connections:
- net GND: now also Q5.2 (S), R5.2
- net VBAT: now also D3.1 (K), LS1.P
- net buzzerPWM: now reaches U3.18 (PB0)
- net buzzerPWM: now also R8.2
- new net: D3.2 (A), LS1.N, Q5.3 (D)
- new net: Q5.1 (G), R5.1, R8.1
- no-connect marks 31 -> 30
